Commit message: use GPU accelerate 3D laser and update the launch file
Signed-off-by: jiajun.liu <jiajun.liu@szkwrobot.com>

File: openni_camera/openni_description/model/kinect.urdf.xacro (robot description, xacro)
@@ -11,5 +11,5 @@
     <link name="camera_rgb_frame"/>
     <joint name="camera_rgb_optical_joint" type="fixed">
-      <origin xyz="0 0 0" rpy="${-M_PI/2} 0 ${-M_PI/2}" />
+      <origin xyz="0 0 0" rpy="${-pi/2} 0 ${-pi/2}" />
       <parent link="camera_rgb_frame" />
       <child link="camera_rgb_optical_frame" />
@@ -23,5 +23,5 @@
       <link name="camera_link">
       <visual>
-       <origin xyz="0 0 0" rpy="0 0 ${M_PI/2}"/>
+       <origin xyz="0 0 0" rpy="0 0 ${pi/2}"/>
         <geometry>
          <mesh filename="package://openni_description/mesh/kinect.dae"/>
@@ -52,5 +52,5 @@
 	<link name="camera_depth_frame"/>
 	<joint name="camera_depth_optical_joint" type="fixed">
-	  <origin xyz="0 0 0" rpy="${-M_PI/2} 0 ${-M_PI/2}" />
+	  <origin xyz="0 0 0" rpy="${-pi/2} 0 ${-pi/2}" />
 	  <parent link="camera_depth_frame" />
 	  <child link="camera_depth_optical_frame" />
@@ -58,5 +58,5 @@
 	<link name="camera_depth_optical_frame"/>
 	<!-- Kinect sensor for simulation -->
-	<sim_3dsensor_kinect/>
+	<xacro:sim_3dsensor_kinect/>
   </xacro:macro>
 </robot>

File: openni_camera/openni_description/model/kinect_gazebo.urdf.xacro (robot description, xacro)
@@ -8,5 +8,5 @@
         <update_rate>20.0</update_rate>
         <camera>
-          <horizontal_fov>${60.0*M_PI/180.0}</horizontal_fov>
+          <horizontal_fov>${60.0*pi/180.0}</horizontal_fov>
           <image>
             <format>B8G8R8</format>

File: turtlebot3/turtlebot3_description/urdf/mlbot.gazebo.xacro (robot description, xacro)
@@ -201,5 +201,5 @@
     <parent link="base_link"/>
     <child link="base_2dscan"/>
-    <origin xyz="0.0 0 0.20" rpy="0 0 0"/>
+    <origin xyz="0.0 0 0.23" rpy="0 0 0"/>
   </joint>
   <link name="base_2dscan">
@@ -377,5 +377,5 @@
   <!-- add laser simulation plugines adaptored for rplidar A1M8 -->
   <gazebo reference="velodyne">
-    <sensor type="ray" name="velodyne-VLP16">      <!-- ray   -->   <!-- gpu_ray -->
+    <sensor type="gpu_ray" name="velodyne-VLP16">
       <pose>0 0 0 0 0 0</pose>
       <visualize>false</visualize>
@@ -386,12 +386,12 @@
             <samples>1875</samples>
             <resolution>1</resolution>
-            <min_angle>0.9</min_angle>
-            <max_angle>130</max_angle>
+            <min_angle>0.0</min_angle>
+            <max_angle>6.28</max_angle>
           </horizontal>
           <vertical>
             <samples>16</samples>
-            <resolution>1</resolution>
-            <min_angle>-0.26</min_angle>   <!-- 15 -->
-            <max_angle> 0.26</max_angle>
+            <resolution>2</resolution>
+            <min_angle> -0.52 </min_angle>
+            <max_angle> 0.52</max_angle>
           </vertical>
         </scan>
@@ -407,5 +407,5 @@
         </noise>
       </ray>
-      <plugin name="gazebo_ros_laser_controller" filename="libgazebo_ros_velodyne_laser.so">     <!-- libgazebo_ros_velodyne_gpu_laser  --> <!-- libgazebo_ros_velodyne_laser  -->
+      <plugin name="gazebo_ros_laser_controller2" filename="libgazebo_ros_velodyne_gpu_laser.so">
         <topicName>/velodyne_points</topicName>
         <frameName>velodyne</frameName>

File: turtlebot3/turtlebot3_description/urdf/mlbot.urdf.xacro (robot description, xacro)
@@ -2,3 +2,7 @@
 <robot name="mlbot" xmlns:xacro="http://ros.org/wiki/xacro">
   <xacro:include filename="$(find turtlebot3_description)/urdf/mlbot.gazebo.xacro"/>
+   <xacro:include filename="$(find openni_description)/model/kinect.urdf.xacro" />
+  <xacro:sensor_kinect parent="base_link"
+  cam_px="0" cam_py="0" cam_pz="0.3"
+  cam_or="0" cam_op="0" cam_oy="0" />
 </robot>
